Commit message: switch to rl modified ver of Nate's fork

File: puppersim/data/pupper_v2a.urdf (robot description, URDF)
Before this commit: robot pupper_v2_dji, 17 links, 16 joints
Links:
- link leftFrontLeg: mass 0.20000 -> 0.106; geometry collision cylinder length=0.075 radius=0.015; visual mesh filename=meshes/Hip_L.obj scale=1.0 1.0 1.0
- link leftFrontLowerLeg: mass 0.10000 -> 0.038; geometry collision box size=0.00951 0.012 0.10758; visual mesh filename=meshes/Lower_Leg_L.obj scale=1.0 1.0 1.0
- link leftFrontToe: mass 0.010000 -> 0.0001; geometry collision sphere radius=0.0095; visual sphere radius=0.01
- link leftFrontUpperLeg: mass 0.20000 -> 0.142; geometry collision cylinder length=0.065 radius=0.015; visual mesh filename=meshes/Upper_Leg_-_Pupper_2.1_v57.obj scale=1.0 1.0 1.0
- link leftRearLeg: mass 0.20000 -> 0.106; geometry collision cylinder length=0.075 radius=0.015; visual mesh filename=meshes/Hip_L.obj scale=1.0 1.0 1.0
- link leftRearLowerLeg: mass 0.10000 -> 0.038; geometry collision box size=0.00951 0.012 0.10758; visual mesh filename=meshes/Lower_Leg_L.obj scale=1.0 1.0 1.0
- link leftRearToe: mass 0.010000 -> 0.0001; geometry collision sphere radius=0.0095; visual sphere radius=0.01
- link leftRearUpperLeg: mass 0.20000 -> 0.142; geometry collision cylinder length=0.065 radius=0.015; visual mesh filename=meshes/Upper_Leg_-_Pupper_2.1_v57.obj scale=1.0 1.0 1.0
- link pupper_v2_dji_chassis: mass 1.00000 -> 0.991; geometry collision mesh filename=meshes/Cube.003.obj scale=1.0 1.0 1.0; visual mesh filename=meshes/Body_Assembly_v3.obj scale=1.0 1.0 1.0
- link rightFrontLeg: mass 0.20000 -> 0.106; geometry collision cylinder length=0.075 radius=0.015; visual mesh filename=meshes/Hip_R.obj scale=1.0 1.0 1.0
- link rightFrontLowerLeg: mass 0.10000 -> 0.038; geometry collision box size=0.00953 0.012 0.10758; visual mesh filename=meshes/Lower_Leg_R.obj scale=1.0 1.0 1.0
- link rightFrontToe: mass 0.010000 -> 0.0001; geometry collision sphere radius=0.0095; visual sphere radius=0.01
- link rightFrontUpperLeg: mass 0.20000 -> 0.142; geometry collision cylinder length=0.065 radius=0.015; visual mesh filename=meshes/Upper_Leg_-_Pupper_2.1_v57.obj scale=1.0 1.0 1.0
- link rightRearLeg: mass 0.20000 -> 0.106; geometry collision cylinder length=0.075 radius=0.015; visual mesh filename=meshes/Hip_R.obj scale=1.0 1.0 1.0
- link rightRearLowerLeg: mass 0.10000 -> 0.038; geometry collision box size=0.00953 0.012 0.10758; visual mesh filename=meshes/Lower_Leg_R.obj scale=1.0 1.0 1.0
- link rightRearToe: mass 0.01 -> 0.0001; geometry collision sphere radius=0.0095; visual sphere radius=0.01
- link rightRearUpperLeg: mass 0.20000 -> 0.142; geometry collision cylinder length=0.065 radius=0.015; visual mesh filename=meshes/Upper_Leg_-_Pupper_2.1_v57.obj scale=1.0 1.0 1.0
Joints:
- joint leftFrontLegMotor: axis 0.00000 -1.00000 0.00000 -> 0 -1.0 0; limit lower=-0.2 upper=.2 effort=100 velocity=100 -> lower=-0.7854 upper=0.7854 effort=0 velocity=0; origin xyz=0.04645 -0.06686 0.00483 rpy=0.00000 -0.00000 0.00000 -> xyz=0.047 -0.1015 0 rpy=0 0 0
- joint leftFrontLowerLegMotor: axis 1.00000 0.00000 0.00000 -> -1.0 0 0; limit lower=-2.4 upper=-.5 effort=100 velocity=100 -> lower=-2.87979 upper=2.87979 effort=0 velocity=0; origin xyz=0.00000 0.00000 -0.08000 rpy=0.00000 -0.00000 0.00000 -> xyz=-0.004 0 -0.08 rpy=0 0 3.14159
- joint leftFrontToe: axis 1.00000 0.00000 0.00000 -> (none); origin xyz=0.0094 0.00000 -0.11000 rpy=0.00000 -0.00000 0.00000 -> xyz=0.002 0 -0.11 rpy=0 0 -3.14159; type fixed -> floating
- joint leftFrontUpperLegMotor: axis 1.00000 0.00000 0.00000 -> 1.0 0 0; limit lower=0.0 upper=.8 effort=100 velocity=100 -> lower=-1.309 upper=4.45059 effort=0 velocity=0; origin xyz=0.02500 0.02000 -0.00500 rpy=0.00000 -0.00000 0.00000 -> xyz=0.0395 0.0265 0 rpy=0 0 0
- joint leftRearLegMotor: axis 0.00000 -1.00000 0.00000 -> 0 -1.0 0; limit lower=-0.2 upper=.2 effort=100 velocity=100 -> lower=-0.7854 upper=0.7854 effort=0 velocity=0; origin xyz=0.04645 0.13313 0.00483 rpy=0.00000 -0.00000 0.00000 -> xyz=0.047 0.0985 0 rpy=0 0 0
- joint leftRearLowerLegMotor: axis 1.00000 0.00000 0.00000 -> -1.0 0 0; limit lower=-2.4 upper=-.5 effort=100 velocity=100 -> lower=-2.87979 upper=2.87979 effort=0 velocity=0; origin xyz=0.00000 0.00000 -0.08000 rpy=0.00000 -0.00000 0.00000 -> xyz=-0.004 0 -0.08 rpy=0 0 3.14159
- joint leftRearToe: axis 1.00000 0.00000 0.00000 -> (none); origin xyz=0.0094 0.00000 -0.11000 rpy=0.00000 -0.00000 0.00000 -> xyz=0.002 0 -0.11 rpy=0 0 -3.14159; type fixed -> floating
- joint leftRearUpperLegMotor: axis 1.00000 0.00000 0.00000 -> 1.0 0 0; limit lower=0.0 upper=.8 effort=100 velocity=100 -> lower=-1.309 upper=4.45059 effort=0 velocity=0; origin xyz=0.02500 0.02000 -0.00500 rpy=0.00000 -0.00000 0.00000 -> xyz=0.0395 0.0265 0 rpy=0 0 0
- joint rightFrontLegMotor: axis 0.00000 -1.00000 0.00000 -> 0 1.0 0; limit lower=-0.2 upper=.2 effort=100 velocity=100 -> lower=-0.7854 upper=0.7854 effort=0 velocity=0; origin xyz=-0.04645 -0.06686 0.00483 rpy=0.00000 -0.00000 0.00000 -> xyz=-0.047 -0.103 0 rpy=0 0 -3.14159
- joint rightFrontLowerLegMotor: axis 1.00000 0.00000 0.00000 -> -1.0 0 0; limit lower=-2.4 upper=-.5 effort=100 velocity=100 -> lower=-2.87979 upper=2.87979 effort=0 velocity=0; origin xyz=0.00000 0.00000 -0.08000 rpy=0.00000 -0.00000 0.00000 -> xyz=-0.004 0 -0.08 rpy=0 0 0
- joint rightFrontToe: axis 1.00000 0.00000 0.00000 -> (none); origin xyz=-0.0094 0.00000 -0.11000 rpy=0.00000 -0.00000 0.00000 -> xyz=-0.002 0 -0.11 rpy=0 0 3.14159; type fixed -> floating
- joint rightFrontUpperLegMotor: axis 1.00000 0.00000 0.00000 -> -1.0 0 0; limit lower=0.0 upper=.8 effort=100 velocity=100 -> lower=-1.309 upper=4.45059 effort=0 velocity=0; origin xyz=-0.02500 0.02000 -0.00500 rpy=0.00000 -0.00000 0.00000 -> xyz=0.0395 -0.028 0 rpy=0 0 0
- joint rightRearLegMotor: axis 0.00000 -1.00000 0.00000 -> 0 1.0 0; limit lower=-0.2 upper=.2 effort=100 velocity=100 -> lower=-0.7854 upper=0.7854 effort=0 velocity=0; origin xyz=-0.04645 0.13313 0.00483 rpy=0.00000 -0.00000 0.00000 -> xyz=-0.047 0.097 0 rpy=0 0 -3.14159
- joint rightRearLowerLegMotor: axis 1.00000 0.00000 0.00000 -> -1.0 0 0; limit lower=-2.4 upper=-.5 effort=100 velocity=100 -> lower=-2.87979 upper=2.87979 effort=0 velocity=0; origin xyz=0.00000 0.00000 -0.08000 rpy=0.00000 -0.00000 0.00000 -> xyz=-0.004 0 -0.08 rpy=0 0 0
- joint rightRearToe: axis 1.00000 0.00000 0.00000 -> (none); origin xyz=-0.0094 0.00000 -0.11000 rpy=0.00000 -0.00000 0.00000 -> xyz=-0.002 0 -0.11 rpy=0 0 3.14159; type fixed -> floating
- joint rightRearUpperLegMotor: axis 1.00000 0.00000 0.00000 -> -1.0 0 0; limit lower=0.0 upper=.8 effort=100 velocity=100 -> lower=-1.309 upper=4.45059 effort=0 velocity=0; origin xyz=-0.02500 0.02000 -0.00500 rpy=0.00000 -0.00000 0.00000 -> xyz=0.0395 -0.028 0 rpy=0 0 0

File: puppersim/data/pupper_v2b.urdf (robot description, URDF)
Before this commit: robot pupper_v2_dji, 17 links, 16 joints
Links:
- link leftFrontLeg: mass 0.50000 -> 0.106; geometry collision cylinder length=0.075 radius=0.015
- link leftFrontLowerLeg: mass 0.10000 -> 0.038; geometry collision box size=0.00951 0.012 0.10758
- link leftFrontToe: mass 0.010000 -> 0.0001; geometry collision sphere radius=0.0095; visual sphere radius=0.01
- link leftFrontUpperLeg: mass 0.20000 -> 0.142; geometry collision cylinder length=0.065 radius=0.015
- link leftRearLeg: mass 0.50000 -> 0.106; geometry collision cylinder length=0.075 radius=0.015
- link leftRearLowerLeg: mass 0.10000 -> 0.038; geometry collision box size=0.00951 0.012 0.10758
- link leftRearToe: mass 0.010000 -> 0.0001; geometry collision sphere radius=0.0095; visual sphere radius=0.01
- link leftRearUpperLeg: mass 0.20000 -> 0.142; geometry collision cylinder length=0.065 radius=0.015
- link pupper_v2_dji_chassis: mass 1.00000 -> 0.991; geometry collision mesh filename=meshes/Cube.003.obj scale=1.0 1.0 1.0
- link rightFrontLeg: mass 0.50000 -> 0.106; geometry collision cylinder length=0.075 radius=0.015
- link rightFrontLowerLeg: mass 0.10000 -> 0.038; geometry collision box size=0.00953 0.012 0.10758
- link rightFrontToe: mass 0.010000 -> 0.0001; geometry collision sphere radius=0.0095; visual sphere radius=0.01
- link rightFrontUpperLeg: mass 0.20000 -> 0.142; geometry collision cylinder length=0.065 radius=0.015
- link rightRearLeg: mass 0.50000 -> 0.106; geometry collision cylinder length=0.075 radius=0.015
- link rightRearLowerLeg: mass 0.10000 -> 0.038; geometry collision box size=0.00953 0.012 0.10758
- link rightRearToe: mass 0.01 -> 0.0001; geometry collision sphere radius=0.0095; visual sphere radius=0.01
- link rightRearUpperLeg: mass 0.20000 -> 0.142; geometry collision cylinder length=0.065 radius=0.015
Joints:
- joint leftFrontLegMotor: axis 0.00000 -1.00000 0.00000 -> 0 -1.0 0; limit (none) -> lower=-0.7854 upper=0.7854 effort=0 velocity=0; origin xyz=0.04645 -0.06686 0.00483 rpy=0.00000 -0.00000 0.00000 -> xyz=0.047 -0.1015 0 rpy=0 0 0; type continuous -> revolute
- joint leftFrontLowerLegMotor: axis 1.00000 0.00000 0.00000 -> -1.0 0 0; limit (none) -> lower=-2.87979 upper=2.87979 effort=0 velocity=0; origin xyz=0.00000 0.00000 -0.08000 rpy=0.00000 -0.00000 0.00000 -> xyz=-0.004 0 -0.08 rpy=0 0 3.14159; type continuous -> revolute
- joint leftFrontToe: axis 1.00000 0.00000 0.00000 -> (none); origin xyz=0.0094 0.00000 -0.11000 rpy=0.00000 -0.00000 0.00000 -> xyz=0.002 0 -0.11 rpy=0 0 -3.14159; type fixed -> floating
- joint leftFrontUpperLegMotor: axis 1.00000 0.00000 0.00000 -> 1.0 0 0; limit (none) -> lower=-1.309 upper=4.45059 effort=0 velocity=0; origin xyz=0.02500 0.02000 -0.00500 rpy=0.00000 -0.00000 0.00000 -> xyz=0.0395 0.0265 0 rpy=0 0 0; type continuous -> revolute
- joint leftRearLegMotor: axis 0.00000 -1.00000 0.00000 -> 0 -1.0 0; limit (none) -> lower=-0.7854 upper=0.7854 effort=0 velocity=0; origin xyz=0.04645 0.13313 0.00483 rpy=0.00000 -0.00000 0.00000 -> xyz=0.047 0.0985 0 rpy=0 0 0; type continuous -> revolute
- joint leftRearLowerLegMotor: axis 1.00000 0.00000 0.00000 -> -1.0 0 0; limit (none) -> lower=-2.87979 upper=2.87979 effort=0 velocity=0; origin xyz=0.00000 0.00000 -0.08000 rpy=0.00000 -0.00000 0.00000 -> xyz=-0.004 0 -0.08 rpy=0 0 3.14159; type continuous -> revolute
- joint leftRearToe: axis 1.00000 0.00000 0.00000 -> (none); origin xyz=0.0094 0.00000 -0.11000 rpy=0.00000 -0.00000 0.00000 -> xyz=0.002 0 -0.11 rpy=0 0 -3.14159; type fixed -> floating
- joint leftRearUpperLegMotor: axis 1.00000 0.00000 0.00000 -> 1.0 0 0; limit (none) -> lower=-1.309 upper=4.45059 effort=0 velocity=0; origin xyz=0.02500 0.02000 -0.00500 rpy=0.00000 -0.00000 0.00000 -> xyz=0.0395 0.0265 0 rpy=0 0 0; type continuous -> revolute
- joint rightFrontLegMotor: axis 0.00000 1.00000 0.00000 -> 0 1.0 0; limit (none) -> lower=-0.7854 upper=0.7854 effort=0 velocity=0; origin xyz=-0.04645 -0.06686 0.00483 rpy=0.00000 -0.00000 0.00000 -> xyz=-0.047 -0.103 0 rpy=0 0 -3.14159; type continuous -> revolute
- joint rightFrontLowerLegMotor: axis 1.00000 0.00000 0.00000 -> -1.0 0 0; limit (none) -> lower=-2.87979 upper=2.87979 effort=0 velocity=0; origin xyz=0.00000 0.00000 -0.08000 rpy=0.00000 -0.00000 0.00000 -> xyz=-0.004 0 -0.08 rpy=0 0 0; type continuous -> revolute
- joint rightFrontToe: axis 1.00000 0.00000 0.00000 -> (none); origin xyz=-0.0094 0.00000 -0.11000 rpy=0.00000 -0.00000 0.00000 -> xyz=-0.002 0 -0.11 rpy=0 0 3.14159; type fixed -> floating
- joint rightFrontUpperLegMotor: axis 1.00000 0.00000 0.00000 -> -1.0 0 0; limit (none) -> lower=-1.309 upper=4.45059 effort=0 velocity=0; origin xyz=-0.02500 0.02000 -0.00500 rpy=0.00000 -0.00000 0.00000 -> xyz=0.0395 -0.028 0 rpy=0 0 0; type continuous -> revolute
- joint rightRearLegMotor: axis 0.00000 1.00000 0.00000 -> 0 1.0 0; limit (none) -> lower=-0.7854 upper=0.7854 effort=0 velocity=0; origin xyz=-0.04645 0.13313 0.00483 rpy=0.00000 -0.00000 0.00000 -> xyz=-0.047 0.097 0 rpy=0 0 -3.14159; type continuous -> revolute
- joint rightRearLowerLegMotor: axis 1.00000 0.00000 0.00000 -> -1.0 0 0; limit (none) -> lower=-2.87979 upper=2.87979 effort=0 velocity=0; origin xyz=0.00000 0.00000 -0.08000 rpy=0.00000 -0.00000 0.00000 -> xyz=-0.004 0 -0.08 rpy=0 0 0; type continuous -> revolute
- joint rightRearToe: axis 1.00000 0.00000 0.00000 -> (none); origin xyz=-0.0094 0.00000 -0.11000 rpy=0.00000 -0.00000 0.00000 -> xyz=-0.002 0 -0.11 rpy=0 0 3.14159; type fixed -> floating
- joint rightRearUpperLegMotor: axis 1.00000 0.00000 0.00000 -> -1.0 0 0; limit (none) -> lower=-1.309 upper=4.45059 effort=0 velocity=0; origin xyz=-0.02500 0.02000 -0.00500 rpy=0.00000 -0.00000 0.00000 -> xyz=0.0395 -0.028 0 rpy=0 0 0; type continuous -> revolute
